Commit message: Gz sim setup

File: urdf/ackerman.xacro (robot description, xacro)
@@ -15,12 +15,12 @@
       <origin rpy="0 0 0" xyz="0 0 0"/>
       <geometry>
-        <mesh filename="package://mentorpiA1_simulator/meshes/acker/base_link.STL"/>
-      </geometry>
-      <material name="black"/>
-    </visual>
-    <collision>
-      <origin rpy="0 0 0" xyz="0 0 0"/>
-      <geometry>
-        <mesh filename="package://mentorpiA1_simulator/meshes/acker/base_link.STL"/>
+        <mesh filename="package://mentorpia1_simulator/meshes/acker/base_link.STL"/>
+      </geometry>
+      <material name="black"/>
+    </visual>
+    <collision>
+      <origin rpy="0 0 0" xyz="0 0 0"/>
+      <geometry>
+        <mesh filename="package://mentorpia1_simulator/meshes/acker/base_link.STL"/>
       </geometry>
     </collision>
@@ -49,12 +49,12 @@
       <origin rpy="0 0 0" xyz="0 0 0"/>
       <geometry>
-        <mesh filename="package://mentorpiA1_simulator/meshes/acker/wheel_lb_Link.STL"/>
-      </geometry>
-      <material name="black"/>
-    </visual>
-    <collision>
-      <origin rpy="0 0 0" xyz="0 0 0"/>
-      <geometry>
-        <mesh filename="package://mentorpiA1_simulator/meshes/acker/wheel_lb_Link.STL"/>
+        <mesh filename="package://mentorpia1_simulator/meshes/acker/wheel_lb_Link.STL"/>
+      </geometry>
+      <material name="black"/>
+    </visual>
+    <collision>
+      <origin rpy="0 0 0" xyz="0 0 0"/>
+      <geometry>
+        <mesh filename="package://mentorpia1_simulator/meshes/acker/wheel_lb_Link.STL"/>
       </geometry>
     </collision>
@@ -75,12 +75,12 @@
       <origin rpy="0 0 0" xyz="0 0 0"/>
       <geometry>
-        <mesh filename="package://mentorpiA1_simulator/meshes/acker/wheel_rb_Link.STL"/>
-      </geometry>
-      <material name="black"/>
-    </visual>
-    <collision>
-      <origin rpy="0 0 0" xyz="0 0 0"/>
-      <geometry>
-        <mesh filename="package://mentorpiA1_simulator/meshes/acker/wheel_rb_Link.STL"/>
+        <mesh filename="package://mentorpia1_simulator/meshes/acker/wheel_rb_Link.STL"/>
+      </geometry>
+      <material name="black"/>
+    </visual>
+    <collision>
+      <origin rpy="0 0 0" xyz="0 0 0"/>
+      <geometry>
+        <mesh filename="package://mentorpia1_simulator/meshes/acker/wheel_rb_Link.STL"/>
       </geometry>
     </collision>
@@ -126,12 +126,12 @@
       <origin rpy="0 0 0" xyz="0 0 0"/>
       <geometry>
-        <mesh filename="package://mentorpiA1_simulator/meshes/acker/wheel_lf_Link.STL"/>
-      </geometry>
-      <material name="black"/>
-    </visual>
-    <collision>
-      <origin rpy="0 0 0" xyz="0 0 0"/>
-      <geometry>
-        <mesh filename="package://mentorpiA1_simulator/meshes/acker/wheel_lf_Link.STL"/>
+        <mesh filename="package://mentorpia1_simulator/meshes/acker/wheel_lf_Link.STL"/>
+      </geometry>
+      <material name="black"/>
+    </visual>
+    <collision>
+      <origin rpy="0 0 0" xyz="0 0 0"/>
+      <geometry>
+        <mesh filename="package://mentorpia1_simulator/meshes/acker/wheel_lf_Link.STL"/>
       </geometry>
     </collision>
@@ -152,12 +152,12 @@
       <origin rpy="0 0 0" xyz="0 0 0"/>
       <geometry>
-        <mesh filename="package://mentorpiA1_simulator/meshes/acker/wheel_rf_Link.STL"/>
-      </geometry>
-      <material name="black"/>
-    </visual>
-    <collision>
-      <origin rpy="0 0 0" xyz="0 0 0"/>
-      <geometry>
-        <mesh filename="package://mentorpiA1_simulator/meshes/acker/wheel_rf_Link.STL"/>
+        <mesh filename="package://mentorpia1_simulator/meshes/acker/wheel_rf_Link.STL"/>
+      </geometry>
+      <material name="black"/>
+    </visual>
+    <collision>
+      <origin rpy="0 0 0" xyz="0 0 0"/>
+      <geometry>
+        <mesh filename="package://mentorpia1_simulator/meshes/acker/wheel_rf_Link.STL"/>
       </geometry>
     </collision>
@@ -179,12 +179,12 @@
       <origin rpy="0 0 0" xyz="0 0 0"/>
       <geometry>
-        <mesh filename="package://mentorpiA1_simulator/meshes/acker/lidar_Link.STL"/>
-      </geometry>
-      <material name="black"/>
-    </visual>
-    <collision>
-      <origin rpy="0 0 0" xyz="0 0 0"/>
-      <geometry>
-        <mesh filename="package://mentorpiA1_simulator/meshes/acker/lidar_Link.STL"/>
+        <mesh filename="package://mentorpia1_simulator/meshes/acker/lidar_Link.STL"/>
+      </geometry>
+      <material name="black"/>
+    </visual>
+    <collision>
+      <origin rpy="0 0 0" xyz="0 0 0"/>
+      <geometry>
+        <mesh filename="package://mentorpia1_simulator/meshes/acker/lidar_Link.STL"/>
       </geometry>
     </collision>
@@ -206,12 +206,12 @@
       <origin rpy="0 0 0" xyz="0 0 0"/>
       <geometry>
-        <mesh filename="package://mentorpiA1_simulator/meshes/acker/cam_Link.STL"/>
-      </geometry>
-      <material name="black"/>
-    </visual>
-    <collision>
-      <origin rpy="0 0 0" xyz="0 0 0"/>
-      <geometry>
-        <mesh filename="package://mentorpiA1_simulator/meshes/acker/cam_Link.STL"/>
+        <mesh filename="package://mentorpia1_simulator/meshes/acker/cam_Link.STL"/>
+      </geometry>
+      <material name="black"/>
+    </visual>
+    <collision>
+      <origin rpy="0 0 0" xyz="0 0 0"/>
+      <geometry>
+        <mesh filename="package://mentorpia1_simulator/meshes/acker/cam_Link.STL"/>
       </geometry>
     </collision>
@@ -224,4 +224,4 @@
   </joint>
   <!-- Include IMU -->
-  <xacro:include filename="$(find mentorpiA1_simulator)/urdf/imu.urdf.xacro"/>
+  <xacro:include filename="$(find mentorpia1_simulator)/urdf/imu.urdf.xacro"/>
 </robot>

File: urdf/mentorpi.xacro (robot description, xacro)
@@ -2,10 +2,5 @@
 <robot name="rosmentor" xmlns:xacro="http://ros.org/wiki/xacro">
     <xacro:property name="machine"      value="$(env MACHINE_TYPE)"/>
-    <xacro:if value="${machine == 'MentorPi_Mecanum'}">
-        <xacro:include filename="$(find mentorpiA1_simulator)/urdf/mecanum.xacro"/>
-    </xacro:if>
-    <xacro:if value="${machine == 'MentorPi_Acker'}">
-        <xacro:include filename="$(find mentorpiA1_simulator)/urdf/ackerman.xacro"/>
-    </xacro:if>
-    <xacro:include filename="$(find mentorpiA1_simulator)/urdf/inertial_matrix.xacro" />
+    <xacro:include filename="$(find mentorpia1_simulator)/urdf/ackerman.xacro"/>
+    <xacro:include filename="$(find mentorpia1_simulator)/urdf/inertial_matrix.xacro" />
 </robot>

Commit message: Fixed pkg naming issues. Sim is portable now. TODO: Modify README.

File: urdf/ackerman.xacro (robot description, xacro)
@@ -15,12 +15,12 @@
       <origin rpy="0 0 0" xyz="0 0 0"/>
       <geometry>
-        <mesh filename="package://mentorpia1_simulator/meshes/acker/base_link.STL"/>
-      </geometry>
-      <material name="black"/>
-    </visual>
-    <collision>
-      <origin rpy="0 0 0" xyz="0 0 0"/>
-      <geometry>
-        <mesh filename="package://mentorpia1_simulator/meshes/acker/base_link.STL"/>
+        <mesh filename="package://mentorpia1_simulator_s2025/meshes/acker/base_link.STL"/>
+      </geometry>
+      <material name="black"/>
+    </visual>
+    <collision>
+      <origin rpy="0 0 0" xyz="0 0 0"/>
+      <geometry>
+        <mesh filename="package://mentorpia1_simulator_s2025/meshes/acker/base_link.STL"/>
       </geometry>
     </collision>
@@ -49,12 +49,12 @@
       <origin rpy="0 0 0" xyz="0 0 0"/>
       <geometry>
-        <mesh filename="package://mentorpia1_simulator/meshes/acker/wheel_lb_Link.STL"/>
-      </geometry>
-      <material name="black"/>
-    </visual>
-    <collision>
-      <origin rpy="0 0 0" xyz="0 0 0"/>
-      <geometry>
-        <mesh filename="package://mentorpia1_simulator/meshes/acker/wheel_lb_Link.STL"/>
+        <mesh filename="package://mentorpia1_simulator_s2025/meshes/acker/wheel_lb_Link.STL"/>
+      </geometry>
+      <material name="black"/>
+    </visual>
+    <collision>
+      <origin rpy="0 0 0" xyz="0 0 0"/>
+      <geometry>
+        <mesh filename="package://mentorpia1_simulator_s2025/meshes/acker/wheel_lb_Link.STL"/>
       </geometry>
     </collision>
@@ -75,12 +75,12 @@
       <origin rpy="0 0 0" xyz="0 0 0"/>
       <geometry>
-        <mesh filename="package://mentorpia1_simulator/meshes/acker/wheel_rb_Link.STL"/>
-      </geometry>
-      <material name="black"/>
-    </visual>
-    <collision>
-      <origin rpy="0 0 0" xyz="0 0 0"/>
-      <geometry>
-        <mesh filename="package://mentorpia1_simulator/meshes/acker/wheel_rb_Link.STL"/>
+        <mesh filename="package://mentorpia1_simulator_s2025/meshes/acker/wheel_rb_Link.STL"/>
+      </geometry>
+      <material name="black"/>
+    </visual>
+    <collision>
+      <origin rpy="0 0 0" xyz="0 0 0"/>
+      <geometry>
+        <mesh filename="package://mentorpia1_simulator_s2025/meshes/acker/wheel_rb_Link.STL"/>
       </geometry>
     </collision>
@@ -126,12 +126,12 @@
       <origin rpy="0 0 0" xyz="0 0 0"/>
       <geometry>
-        <mesh filename="package://mentorpia1_simulator/meshes/acker/wheel_lf_Link.STL"/>
-      </geometry>
-      <material name="black"/>
-    </visual>
-    <collision>
-      <origin rpy="0 0 0" xyz="0 0 0"/>
-      <geometry>
-        <mesh filename="package://mentorpia1_simulator/meshes/acker/wheel_lf_Link.STL"/>
+        <mesh filename="package://mentorpia1_simulator_s2025/meshes/acker/wheel_lf_Link.STL"/>
+      </geometry>
+      <material name="black"/>
+    </visual>
+    <collision>
+      <origin rpy="0 0 0" xyz="0 0 0"/>
+      <geometry>
+        <mesh filename="package://mentorpia1_simulator_s2025/meshes/acker/wheel_lf_Link.STL"/>
       </geometry>
     </collision>
@@ -152,12 +152,12 @@
       <origin rpy="0 0 0" xyz="0 0 0"/>
       <geometry>
-        <mesh filename="package://mentorpia1_simulator/meshes/acker/wheel_rf_Link.STL"/>
-      </geometry>
-      <material name="black"/>
-    </visual>
-    <collision>
-      <origin rpy="0 0 0" xyz="0 0 0"/>
-      <geometry>
-        <mesh filename="package://mentorpia1_simulator/meshes/acker/wheel_rf_Link.STL"/>
+        <mesh filename="package://mentorpia1_simulator_s2025/meshes/acker/wheel_rf_Link.STL"/>
+      </geometry>
+      <material name="black"/>
+    </visual>
+    <collision>
+      <origin rpy="0 0 0" xyz="0 0 0"/>
+      <geometry>
+        <mesh filename="package://mentorpia1_simulator_s2025/meshes/acker/wheel_rf_Link.STL"/>
       </geometry>
     </collision>
@@ -179,12 +179,12 @@
       <origin rpy="0 0 0" xyz="0 0 0"/>
       <geometry>
-        <mesh filename="package://mentorpia1_simulator/meshes/acker/lidar_Link.STL"/>
-      </geometry>
-      <material name="black"/>
-    </visual>
-    <collision>
-      <origin rpy="0 0 0" xyz="0 0 0"/>
-      <geometry>
-        <mesh filename="package://mentorpia1_simulator/meshes/acker/lidar_Link.STL"/>
+        <mesh filename="package://mentorpia1_simulator_s2025/meshes/acker/lidar_Link.STL"/>
+      </geometry>
+      <material name="black"/>
+    </visual>
+    <collision>
+      <origin rpy="0 0 0" xyz="0 0 0"/>
+      <geometry>
+        <mesh filename="package://mentorpia1_simulator_s2025/meshes/acker/lidar_Link.STL"/>
       </geometry>
     </collision>
@@ -206,12 +206,12 @@
       <origin rpy="0 0 0" xyz="0 0 0"/>
       <geometry>
-        <mesh filename="package://mentorpia1_simulator/meshes/acker/cam_Link.STL"/>
-      </geometry>
-      <material name="black"/>
-    </visual>
-    <collision>
-      <origin rpy="0 0 0" xyz="0 0 0"/>
-      <geometry>
-        <mesh filename="package://mentorpia1_simulator/meshes/acker/cam_Link.STL"/>
+        <mesh filename="package://mentorpia1_simulator_s2025/meshes/acker/cam_Link.STL"/>
+      </geometry>
+      <material name="black"/>
+    </visual>
+    <collision>
+      <origin rpy="0 0 0" xyz="0 0 0"/>
+      <geometry>
+        <mesh filename="package://mentorpia1_simulator_s2025/meshes/acker/cam_Link.STL"/>
       </geometry>
     </collision>
@@ -224,4 +224,4 @@
   </joint>
   <!-- Include IMU -->
-  <xacro:include filename="$(find mentorpia1_simulator)/urdf/imu.urdf.xacro"/>
+  <xacro:include filename="$(find mentorpia1_simulator_s2025)/urdf/imu.urdf.xacro"/>
 </robot>

File: urdf/mentorpi.xacro (robot description, xacro)
@@ -2,5 +2,5 @@
 <robot name="rosmentor" xmlns:xacro="http://ros.org/wiki/xacro">
     <xacro:property name="machine"      value="$(env MACHINE_TYPE)"/>
-    <xacro:include filename="$(find mentorpia1_simulator)/urdf/ackerman.xacro"/>
-    <xacro:include filename="$(find mentorpia1_simulator)/urdf/inertial_matrix.xacro" />
+    <xacro:include filename="$(find mentorpia1_simulator_s2025)/urdf/ackerman.xacro"/>
+    <xacro:include filename="$(find mentorpia1_simulator_s2025)/urdf/inertial_matrix.xacro" />
 </robot>

File: urdf/mentorpia1.urdf (robot description, URDF)
Before this commit: robot rosmentor, 13 links, 12 joints
Links:
- link base_link: geometry collision mesh filename=package://mentorpia1_simulator_s2025/meshes/acker/base_link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; visual mesh filename=package://mentorpia1_simulator_s2025/meshes/acker/base_link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
- link depth_cam: geometry collision mesh filename=package://mentorpia1_simulator_s2025/meshes/acker/cam_Link.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; visual mesh filename=package://mentorpia1_simulator_s2025/meshes/acker/cam_Link.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
- link lidar_frame: geometry collision mesh filename=package://mentorpia1_simulator_s2025/meshes/acker/lidar_Lin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; visual mesh filename=package://mentorpia1_simulator_s2025/meshes/acker/lidar_Lin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
- link wheel_lb_Link: geometry collision mesh filename=package://mentorpia1_simulator_s2025/meshes/acker/wheel_lb_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; visual mesh filename=package://mentorpia1_simulator_s2025/meshes/acker/wheel_lb_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
- link wheel_lf_Link: geometry collision mesh filename=package://mentorpia1_simulator_s2025/meshes/acker/wheel_lf_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; visual mesh filename=package://mentorpia1_simulator_s2025/meshes/acker/wheel_lf_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
- link wheel_rb_Link: geometry collision mesh filename=package://mentorpia1_simulator_s2025/meshes/acker/wheel_rb_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; visual mesh filename=package://mentorpia1_simulator_s2025/meshes/acker/wheel_rb_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
- link wheel_rf_Link: geometry collision mesh filename=package://mentorpia1_simulator_s2025/meshes/acker/wheel_rf_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; visual mesh filename=package://mentorpia1_simulator_s2025/meshes/acker/wheel_rf_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
